File: Hardware/Amplifier/INA129-Amplifier/INA129-Amplifier.kicad_sch (KiCad schematic)
At the start: 14 parts, among them U1 INA129, U2 LM7805_TO220

Commit message: Created INA Amplifier Rev1, created outputs for shipped model
Parts:
- removed R4: 47.4k, symbol Device:R
- added C1, C2: 0.2n, symbol Device:C
- added C10, C11, C12, C8: 0.1u, Capacitor_SMD:C_0805_2012Metric, symbol Device:C
- added C7, C9: 10u, Capacitor_THT:CP_Radial_D4.0mm_P2.00mm, symbol Device:C_Polarized
- added H1, H2, H3, H4: MountingHole, MountingHole:MountingHole_3.2mm_M3, symbol Mechanical:MountingHole
- added J1, J2, J3, J4, J5, J6, J7: Conn_01x02, Connector_PinHeader_2.54mm:PinHeader_1x02_P2.54mm_Vertical, symbol Connector_Generic:Conn_01x02
- added J8, J9: Conn_01x01, Connector_PinHeader_2.54mm:PinHeader_1x01_P2.54mm_Vertical, symbol Connector_Generic:Conn_01x01
- added R10: 56, Resistor_THT:R_Axial_DIN0309_L9.0mm_D3.2mm_P12.70mm_Horizontal, symbol Device:R
- added R11, R13, R14: 10k, Resistor_SMD:R_0805_2012Metric, symbol Device:R
- added R12: 2200, Resistor_SMD:R_0805_2012Metric, symbol Device:R
- added R2, R3: 47.4k, Resistor_THT:R_Axial_DIN0309_L9.0mm_D3.2mm_P12.70mm_Horizontal, symbol Device:R
- added R6: 100k, Resistor_THT:R_Axial_DIN0309_L9.0mm_D3.2mm_P12.70mm_Horizontal, symbol Device:R
- added R8, R9: 100k, Resistor_SMD:R_0805_2012Metric, symbol Device:R
- added TP+9V1: TPP9V, TestPoint:TestPoint_Pad_D4.0mm, symbol Connector:TestPoint
- added TP-9V1: TPN9V, TestPoint:TestPoint_Pad_D4.0mm, symbol Connector:TestPoint
- added TPBiasOut1: BuffereBiasddOutput, TestPoint:TestPoint_Pad_D4.0mm, symbol Connector:TestPoint
- added TPBufOut1: Buffered_Output, TestPoint:TestPoint_Pad_D4.0mm, symbol Connector:TestPoint
- added TPGND1: Ground, TestPoint:TestPoint_Pad_D4.0mm, symbol Connector:TestPoint
- added U3: LM358, Package_DIP:DIP-8_W7.62mm_LongPads, symbol Amplifier_Operational:LM358
- C3, C4: footprint (none) -> Capacitor_SMD:C_0805_2012Metric
- C5: renamed from C1; footprint (none) -> Capacitor_SMD:C_0805_2012Metric; now not fitted
- C6: renamed from C2; footprint (none) -> Capacitor_SMD:C_0805_2012Metric; now not fitted
- R1: renamed from R2; footprint (none) -> Resistor_SMD:R_0805_2012Metric
- R4: renamed from R3; footprint (none) -> Resistor_SMD:R_0805_2012Metric
- R5: value 47.4k -> 100k; footprint (none) -> Resistor_THT:R_Axial_DIN0309_L9.0mm_D3.2mm_P12.70mm_Horizontal; now not fitted
- R7: renamed from R1; value 330 -> 56; footprint (none) -> Resistor_SMD:R_0805_2012Metric
- TPE+1: renamed from TP1; footprint (none) -> TestPoint:TestPoint_Pad_D4.0mm
- TPE-1: renamed from TP2; footprint (none) -> TestPoint:TestPoint_Pad_D4.0mm
- TPRawOut1: renamed from TP3; footprint (none) -> TestPoint:TestPoint_Pad_D4.0mm
- U1: footprint Package_DIP:DIP-8_W7.62mm -> Package_DIP:DIP-8_W7.62mm_LongPads
- U2: now not fitted
Connections:
- net +9V: now also C11.1, J3.1 (Pin_1), J3.2 (Pin_2), R11.1, TP+9V1.1, U3.8 (V+)
- net -9V: now also C12.1, J4.1 (Pin_1), J4.2 (Pin_2), TP-9V1.1, U3.4 (V-)
- net GND: now also R5.2, C1.2, C10.1, C11.2, C12.2, C2.1, C9.2, J5.1 (Pin_1), J5.2 (Pin_2), J8.1 (Pin_1), J9.1 (Pin_1), R12.2, R6.1, R8.1, R9.1, TPGND1.1; no longer R5.1
- net NegInput: now reaches R4.1, TPE-1.1
- net NegInput: now also C2.2, J2.1 (Pin_1), J2.2 (Pin_2), R3.1
- net NegInputProtected: now reaches R4.2, U1.2 (-)
- net NegInputProtected: now also R3.2, R6.2, R9.2
- net Gain2: now reaches R7.1, U1.1 (Rg)
- net Gain2: now also R10.1
- net PosInputProtected: now reaches R1.2, U1.3 (+)
- net PosInputProtected: now also R5.1, R2.2, R8.2
- net UnBufferedOutput: now reaches TPRawOut1.1, U1.6
- net UnBufferedOutput: now also U3.3 (+)
- net Gain1: now reaches R7.2, U1.8 (Rg)
- net Gain1: now also R10.2
- net PosInput: now reaches R1.1, TPE+1.1
- net PosInput: now also C1.1, J1.1 (Pin_1), J1.2 (Pin_2), R2.1; no longer R5.2
- new net: C7.1, C8.2, R11.2, R12.1, U3.5 (+)
- new net: C10.2, C9.1, R14.2
- new net: R13.2, R14.1, U3.6 (-)
- new net BufferedOutput: C7.2, C8.1, TPBufOut1.1, U3.1, U3.2 (-)
- new net ConditionedOutput: J6.1 (Pin_1), J6.2 (Pin_2), J7.1 (Pin_1), J7.2 (Pin_2), R13.1, TPBiasOut1.1, U3.7
Other:
- note added: "Grounding resistors are necessary for dc bias stability input protections resistors may not be (could hurt performance) but no conclusive evidence that it is directly harmful"
- note removed: "approx 50k matched Resistors used to reduce electrocution risk and provide bias current path to reduce noise"
- moved on the sheet: C3, C4, R1, R4, R7, TPE+1, TPE-1, TPRawOut1, U1
