File: Hardware/Amplifier/Probe_Amplifier_Rev2/INAAmplifierRev2/INAAmplifierRev2.kicad_pcb (KiCad board)
At the start: 2 copper layers, 99.9 x 49.9 mm, 55 parts, among them J1 Conn_01x02, J10 Conn_01x01, J11 Conn_01x01, J12 Conn_01x04, J13 Conn_01x03, J14 Conn_01x04, J2 Conn_01x02, J3 Conn_01x02, J4 Conn_01x02, J5 Conn_01x02, J6 Conn_01x02, J7 Conn_01x02, J8 Conn_01x02, J9 Conn_01x02, U1 INA129, U2 LM358

Commit message: fixed the INA AMplifer DC Bias Buffer
Parts:
- added C13: 220u, Capacitor_THT:CP_Radial_D6.3mm_P2.50mm, F.Cu at (128.7, 141.0)
- C5: value 1u -> 1.22u
- R12: value 2200 -> 1Meg
- moved R11 27.0 mm to (97.9, 135.4)
- moved TP_DCBIAS1 6.43 mm to (130.9, 133.9)
- moved J4 6.28 mm to (125.3, 132.1), turned to 0 degrees
- moved R12 1.40 mm to (124.8, 141.0)
Connections:
- C5 pad 2: /VbiasOutput -> Net-(U2A-+)
- C6 pad 2: /VbiasOutput -> Net-(U2A-+)
- J4 pad 1: /BiasUnbuffered -> /DC_Bias_Buffer
- J4 pad 2: /BiasUnbuffered -> /DC_Bias_Buffer
- R11 pad 2: /BiasUnbuffered -> Net-(U2A-+)
- R12 pad 1: /BiasUnbuffered -> Net-(U2B-+)
- R12 pad 2: GND -> Net-(U2A-+)
- R13 pad 2: /VbiasOutput -> Net-(U2A-+)
- TP_DCBIAS1 pad 1: /BiasUnbuffered -> /DC_Bias_Buffer
- U2 pad 3: /VbiasOutput -> Net-(U2A-+)
- U2 pad 5: /BiasUnbuffered -> Net-(U2B-+)
- U2 pad 6: /VbiasOutput -> /DC_Bias_Buffer
- U2 pad 7: /VbiasOutput -> /DC_Bias_Buffer
Routing:
- net Net-(U2A-+): track 0.00 -> 40.3 mm
- net /VbiasOutput: track 36.2 -> 0.00 mm
- net GND: track 66.0 -> 89.2 mm
- net /BiasUnbuffered: track 19.4 -> 0.00 mm
- net /DC_Bias_Buffer: track 0.00 -> 16.0 mm
- net +9V: track 92.9 -> 103.4 mm
- net Net-(U2B-+): track 0.00 -> 9.07 mm
Other:
- board text added: "1.6 in."
- board text added: "3.56 in."
- board text added: "Buffered DC Bias"
- board text added: "M3"
- board text removed: "GND, Ref GND"
- board text removed: "Unbuffered DC Bias"

Commit message: Changed power connectors, added film caps, general corrections for rev 2
Parts:
- added C14: 0.1u, Capacitor_THT:C_Rect_L7.2mm_W3.5mm_P5.00mm_FKS2_FKP2_MKS2_MKP2, F.Cu at (87.9, 137.1)
- added J15: Conn_01x02, Connector_PinHeader_2.54mm:PinHeader_1x02_P2.54mm_Vertical, F.Cu at (142.1, 140.5)
- C13: value 220u -> 2.2u
- C5: value 1.22u -> 0.22u
- J13: value Conn_01x03 -> Conn_01x02; footprint Connector_JST:JST_XH_B3B-XH-A_1x03_P2.50mm_Vertical -> Connector_PinHeader_2.54mm:PinHeader_1x02_P2.54mm_Vertical
- R11: value 10k -> 56k
- R12: value 1Meg -> 100k
- R13: value 2.2k -> 12k
- moved C5 5.21 mm to (91.2, 141.9), turned to 180 degrees
- moved R13 3.25 mm to (97.1, 138.4)
- moved R11 2.18 mm to (100.1, 135.4)
- moved J13 2.12 mm to (142.1, 132.8), turned to 0 degrees
Connections:
- C5 pad 1: Net-(C5-Pad1) -> Net-(U2A-+)
- C5 pad 2: Net-(U2A-+) -> Net-(C14-Pad1)
- C6 pad 1: Net-(C5-Pad1) -> Net-(C14-Pad1)
- TPRawOut1 pad 1: Net-(C5-Pad1) -> Net-(C14-Pad1)
- U1 pad 6: Net-(C5-Pad1) -> Net-(C14-Pad1)
Routing:
- net Net-(C14-Pad1): track 0.00 -> 22.6 mm
- net Net-(C5-Pad1): track 18.4 -> 0.00 mm
- net -9V: track 112.1 -> 109.0 mm
- net Net-(U2A-+): track 40.3 -> 43.3 mm
- net +9V: track 103.4 -> 105.5 mm
Other:
- board text added: "+9 GND"
- board text added: "GND -9V"
- board text removed: "+9 GND -9"
