File: Hardware/Amplifier/Probe_Amplifier_Rev2/INAAmplifierRev2/INAAmplifierRev2.kicad_sch (KiCad schematic)
At the start: 60 parts, among them J1 Conn_01x02, J10 Conn_01x01, J11 Conn_01x01, J12 Conn_01x04, J13 Conn_01x03, J14 Conn_01x04, J2 Conn_01x02, J3 Conn_01x02, J4 Conn_01x02, J5 Conn_01x02, J6 Conn_01x02, J7 Conn_01x02, J8 Conn_01x02, J9 Conn_01x02, U1 INA129, U2 LM358, U3 LM7805_TO220

Commit message: fixed the INA AMplifer DC Bias Buffer
Parts:
- added C13: 220u, Capacitor_THT:CP_Radial_D6.3mm_P2.50mm, symbol Device:C_Polarized
- C5: value 1u -> 1.22u
- R12: value 2200 -> 1Meg
Connections:
- net GND: now also C13.2; no longer R12.2
- net BiasUnbuffered renamed DC_Bias_Buffer
- net DC_Bias_Buffer: now also U2.6 (-), U2.7; no longer R11.2, R12.1, U2.5 (+)
- net VbiasOutput: no longer names the net of C5.2, C6.2, R13.2, U2.3 (+)
- net VbiasOutput: now also R11.2, R12.2; no longer U2.6 (-), U2.7
- new net: C13.1, R12.1, U2.5 (+)
Other:
- note added: "LowPass Filter To Tap Off DC Offset"
- note removed: "DC Voltage Bias With Buffer For Output"
- moved on the sheet: C5, C6, R13, TPRawOut1

Commit message: Changed power connectors, added film caps, general corrections for rev 2
Parts:
- removed J13: Conn_01x03, Connector_JST:JST_XH_B3B-XH-A_1x03_P2.50mm_Vertical, symbol Connector_Generic:Conn_01x03
- added C14: 0.1u, Capacitor_THT:C_Rect_L7.2mm_W3.5mm_P5.00mm_FKS2_FKP2_MKS2_MKP2, symbol Device:C
- added J13, J15: Conn_01x02, Connector_PinHeader_2.54mm:PinHeader_1x02_P2.54mm_Vertical, symbol Connector_Generic:Conn_01x02
- C13: value 220u -> 2.2u
- C5: value 1.22u -> 0.22u; now not fitted
- R11: value 10k -> 56k
- R12: value 1Meg -> 100k
- R13: value 2.2k -> 12k
Connections:
- net +9V: now also J13.1 (Pin_1)
- net -9V: now also J15.2 (Pin_2)
- net GND: now also J13.2 (Pin_2), J15.1 (Pin_1)
- net at C6.2, R11.2, R12.2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: now also C5.1, C14.2; no longer C5.2
- net at C6.1, TPRawOut1.1, U1.6: now also C5.2, C14.1; no longer C5.1
