File: PresentationMaterial/HardwareForImages/Rev2AmplifierForImageTaking/_autosave-Rev2AmplifierForImageTaking.kicad_sch (KiCad schematic)
At the start: 48 parts, among them J10 Conn_01x01, J11 Conn_01x01, J12 Conn_01x04, J13 Conn_01x02, J14 Conn_01x04, J15 Conn_01x02, J4 Conn_01x02, J5 Conn_01x02, J7 Conn_01x02, J8 Conn_01x02, J9 Conn_01x02, U1 INA129, U2 LM358, U3 LM7805_TO220

Commit message: Added a preliminary block diagram to powerpoint
Connections:
- net at C1.2, R11.2, R13.2: now also R12.2, U2.3 (+)
Changed lines of the file:
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@@
+	)
+	(junction
+		(at 162.56 99.06)
+		(diameter 0)
+		(color 0 0 0 0)
 	)
 	(junction
@@
 		)
 		(stroke
+			(width 0)
+			(type default)
+		)
+	)
+	(wire
+		(pts
+			(xy 137.16 99.06) (xy 162.56 99.06)
+		)
+		(stroke
